Commit message: system update backup

File: src/abb_irb4600_60_205_moveit_config/config/abb_irb4600_60_205.ros2_control.xacro (robot description, xacro)
@@ -2,9 +2,9 @@
 <robot xmlns:xacro="http://www.ros.org/wiki/xacro">
     <xacro:macro name="abb_irb4600_60_205_ros2_control" params="name initial_positions_file">
-        <xacro:property name="initial_positions" value="${xacro.load_yaml(initial_positions_file)['initial_positions']}"/>
+        <xacro:property name="initial_positions" value="${load_yaml(initial_positions_file)['initial_positions']}"/>
         <ros2_control name="${name}" type="system">
             <hardware>
                 <!-- By default, set up controllers for simulation. This won't work on real hardware -->
-                <plugin>gz_ros2_control/GazeboSimSystem</plugin>
+                <plugin>mock_components/GenericSystem</plugin>
             </hardware>
             <joint name="joint_1">

File: src/abb_irb4600_60_205_moveit_config/config/abb_irb4600_60_205.urdf.xacro (robot description, xacro)
@@ -6,4 +6,4 @@
     <!-- Import control_xacro -->
     <xacro:include filename="abb_irb4600_60_205.ros2_control.xacro" />
-    <xacro:abb_irb4600_60_205_ros2_control name="GazeboSimSystem" initial_positions_file="$(arg initial_positions_file)"/>
+    <xacro:abb_irb4600_60_205_ros2_control name="FakeSystem" initial_positions_file="$(arg initial_positions_file)"/>
 </robot>

File: src/warehouse_manage/models/abb_irb4600_60_205.urdf (robot description, URDF)
Before this commit: robot abb_irb4600_60_205, 10 links, 9 joints
Links:
- added link caster, mass 1; collision sphere radius=0.2; visual sphere radius=0.2
- added link caster_pitch, mass 0.01; collision sphere radius=0.01; visual sphere radius=0.01
- added link caster_roll, mass 0.01; collision sphere radius=0.01; visual sphere radius=0.01
- added link chassis, mass 10.0; collision box size=2.0 1.0 0.5; visual box size=2.0 1.0 0.5
- added link left_wheel, mass 1; collision cylinder length=0.2 radius=0.4; visual cylinder length=0.2 radius=0.4
- added link right_wheel, mass 1; collision cylinder length=0.2 radius=0.4; visual cylinder length=0.2 radius=0.4
- link base_link: mass 1.0 -> 10.0
Joints:
- added joint caster_pitch_joint: type revolute, parent chassis, child caster_pitch, origin xyz=0.8 0 -0.2 rpy=0 0 0, axis 1 0 0, limit lower=-1.79769e+308 upper=1.79769e+308 effort=50 velocity=5
- added joint caster_roll_joint: type revolute, parent caster_pitch, child caster_roll, origin xyz=0 0 0, axis 0 1 0, limit lower=-1.79769e+308 upper=1.79769e+308 effort=50 velocity=5
- added joint caster_spin_joint: type revolute, parent caster_roll, child caster, origin xyz=0 0 0, axis 0 0 1, limit lower=-1.79769e+308 upper=1.79769e+308 effort=50 velocity=5
- added joint chassis_to_base: type fixed, parent chassis, child base_link, origin xyz=0 0 0.25 rpy=0 0 0
- added joint left_wheel_joint: type revolute, parent chassis, child left_wheel, origin xyz=-0.5 0.6 0 rpy=-1.5707 0 0, axis 0 0 1, limit lower=-1.79769e+308 upper=1.79769e+308 effort=1000.0 velocity=30.0
- added joint right_wheel_joint: type revolute, parent chassis, child right_wheel, origin xyz=-0.5 -0.6 0 rpy=-1.5707 0 0, axis 0 0 1, limit lower=-1.79769e+308 upper=1.79769e+308 effort=1000.0 velocity=30.0
- joint joint_1: limit lower=-3.141 upper=3.141 effort=0 velocity=3.054 -> lower=-15.0 upper=15.0 effort=1000.0 velocity=30.0
- joint joint_2: limit lower=-1.570 upper=2.617 effort=0 velocity=3.054 -> lower=-15.0 upper=15.0 effort=1000.0 velocity=30.0
- joint joint_3: limit lower=-3.141 upper=1.308 effort=0 velocity=3.054 -> lower=-15.0 upper=15.0 effort=1000.0 velocity=30.0
- joint joint_4: limit lower=-6.981 upper=6.981 effort=0 velocity=4.363 -> lower=-15.0 upper=15.0 effort=1000.0 velocity=30.0
- joint joint_5: limit lower=-2.181 upper=2.094 effort=0 velocity=4.363 -> lower=-15.0 upper=15.0 effort=1000.0 velocity=30.0
- joint joint_6: limit lower=-6.981 upper=6.981 effort=0 velocity=6.283 -> lower=-15.0 upper=15.0 effort=1000.0 velocity=30.0

Commit message: before add two robots

File: src/abb_irb4600_60_205_moveit_config/config/abb_irb4600_60_205.ros2_control.xacro (robot description, xacro)
@@ -2,5 +2,5 @@
 <robot xmlns:xacro="http://www.ros.org/wiki/xacro">
     <xacro:macro name="abb_irb4600_60_205_ros2_control" params="name initial_positions_file">
-        <xacro:property name="initial_positions" value="${load_yaml(initial_positions_file)['initial_positions']}"/>
+        <xacro:property name="initial_positions" value="${xacro.load_yaml(initial_positions_file)['initial_positions']}"/>
         <ros2_control name="${name}" type="system">
             <hardware>

File: src/abb_irb4600_60_205_moveit_config/config/abb_irb4600_60_205.urdf.xacro (robot description, xacro)
@@ -3,5 +3,5 @@
     <xacro:arg name="initial_positions_file" default="initial_positions.yaml" />
     <!-- Import abb_irb4600_60_205 urdf file -->
-    <xacro:include filename="$(find warehouse_manage)/models/abb_irb4600_60_205.urdf" />
+    <xacro:include filename="$(find warehouse_manage)/models/abb_irb4600_60_205/model.urdf" />
     <!-- Import control_xacro -->
     <xacro:include filename="abb_irb4600_60_205.ros2_control.xacro" />

File: src/warehouse_manage/models/abb_irb4600_60_205/model.urdf (robot description, URDF)
Before this commit: robot abb_irb4600_60_205, 16 links, 15 joints
Links:
- removed link base
- removed link caster
- removed link caster_pitch
- removed link caster_roll
- removed link chassis
- removed link left_wheel
- removed link right_wheel
Joints:
- removed joint base_link-base
- removed joint caster_pitch_joint
- removed joint caster_roll_joint
- removed joint caster_spin_joint
- removed joint chassis_to_base
- removed joint left_wheel_joint
- removed joint right_wheel_joint
